File: Eagle/EARS.sch (EAGLE design)
At the start: 23 parts, among them J1 1X2-3.5MM, J2 CORTEX_DEBUG_SMD, X1 ECX_34G

Commit message: Fixed schematics, added sense circuitry, added solenoid switch circuitry.  Finished layout Rev 1.1
Parts:
- added C8: 10u, rcl:C-EUC0603
- added D2: BAS40, diode:BAS40
- added IC1: LM386MM-1, linear:LM386MM-1
- added JP3: (no value), pinhead:PINHD-1X2
- added Q1: IRLb8721, adafruit:MOSFET-NGDS_TO220V
- added R3: 28k, rcl:R-US_R0603
- added R4: 0, rcl:R-US_R0603
- added R5: 1k, rcl:R-US_R0603
- added R6: 10k, rcl:R-US_R0603
- JP2: device pinhead:PINHD-1X8 -> pinhead:PINHD-1X4
Connections:
- removed net P_IN1: JP2.5, U$1.PA5
- removed net P_IN2: JP2.6, U$1.PA6
- removed net P_IN3: JP2.7, U$1.PA7
- removed net P_IN4: JP2.8, U$1.PB0
- removed net P_OUT1: JP2.1, U$1.PA1
- removed net P_OUT2: JP2.2, U$1.PA2
- removed net P_OUT3: JP2.3, U$1.PA3
- removed net P_OUT4: JP2.4, U$1.PA4
- removed net SOL_1: JP1.2, U$1.PB13
- removed net SOL_2: JP1.3, U$1.PB14
- new net AGND: JP1.3, JP1.4, R3.1, R4.1
- new net FB: IC1.-IN, R5.2, R6.1
- new net FLYBACK: D2.A, R3.2
- new net NPN: JP1.1, JP1.2, Q1.S
- new net NPN_DRV: Q1.G, U$1.PB5
- new net NRST: JP3.2, U$1.NRST
- new net PRESSURE: IC1.OUT, R6.2, U$1.PA4
- new net PRSR_IN: JP2.3, R5.1
- net 12V: now also D2.C, Q1.D; no longer JP1.1
- net 3V3: now also C8.2, IC1.VS, JP2.1
- net GND: now also C8.1, IC1.+IN, IC1.GND, JP2.2, JP2.4, JP3.1, R4.2; no longer JP1.4
Other:
- moved on the sheet: JP1

Commit message: Fixed Silk Screen
Parts:
- renumbered IC1 to U3, U$1 to U1, U$2 to U2
